File: pcb/idawgz32/idawgz32.kicad_pcb (KiCad board)
At the start: 2 copper layers, 98.7 x 45.5 mm, 83 parts, among them J1 USB_C_Receptacle_USB2.0, SW1 SW_Push, SW10 SW_Push, SW11 SW_Push, SW12 SW_Push, SW13 SW_Push, SW14 SW_Push, SW15 SW_Push, SW16 SW_Push, SW17 SW_Push, SW18 SW_Push, SW19 SW_Push, SW2 SW_Push, SW20 SW_Push, SW21 SW_Push, SW22 SW_Push, SW23 SW_Push, SW24 SW_Push, SW25 SW_Push, SW26 SW_Push, SW27 SW_Push, SW28 SW_Push, SW29 SW_Push, SW3 SW_Push, SW30 SW_Push, SW31 SW_Push, SW32 SW_Push, SW4 SW_Push, SW41 BOOT, SW42 RESET, SW5 SW_Push, SW6 SW_Push, SW7 SW_Push, SW8 SW_Push, SW9 SW_Push, U1 CH552T, U2 USBLC6-2SC6

Commit message: update gerbers
Parts:
- removed F1: 500mA, Fuse:Fuse_0402_1005Metric
- removed U2: USBLC6-2SC6, Package_TO_SOT_SMD:SOT-23-6
- moved C2 7.29 mm to (77.2, 53.2), turned to 180 degrees
- moved C1 7.05 mm to (79.7, 53.9)
- moved R4 6.05 mm to (81.2, 40.9)
- moved R1 5.83 mm to (79.0, 61.9)
- moved SW24 5.78 mm to (95.7, 63.6)
- moved SW27 5.78 mm to (43.7, 69.9)
- moved D7 5.78 mm to (63.8, 42.7), turned to 165 degrees
- moved D29 5.78 mm to (53.5, 67.9), turned to 165 degrees
- moved SW32 5.78 mm to (89.4, 74.6)
- moved SW6 5.78 mm to (99.8, 43.8)
- moved J1 5.78 mm to (75.2, 40.3)
- moved SW21 5.78 mm to (46.0, 61.2)
- moved SW1 5.78 mm to (33.3, 39.2)
- moved SW5 5.78 mm to (50.7, 43.8)
- moved D10 5.78 mm to (118.3, 43.5)
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Connections:
- C1 pad 1: VCC -> VBUS
- J1 pad A6: PORT+ -> UDP
- J1 pad A7: PORT- -> UDM
- J1 pad B6: PORT+ -> UDP
- J1 pad B7: PORT- -> UDM
- U1 pad 1: P3.2_A3 -> col1
- U1 pad 10: P3.0_RX -> row4
- U1 pad 11: P3.3 -> col10
- U1 pad 12: P3.4 -> col9
- U1 pad 13: P3.5 -> col8
- U1 pad 16: P1.3 -> col7
- U1 pad 17: P1.2 -> col6
- U1 pad 19: VCC -> VBUS
- U1 pad 2: P1.4_CS -> col2
- U1 pad 3: P1.5_MOSI -> col3
- U1 pad 4: P1.6_MISO -> col4
- U1 pad 5: P1.7_SCK -> col5
- U1 pad 7: P1.0 -> row1
- U1 pad 8: P1.1_A0 -> row2
- U1 pad 9: P3.1_TX -> row3
Routing:
- net GND: track 0.00 -> 178.4 mm, vias 0 -> 1
- net row2: track 0.00 -> 109.5 mm, vias 0 -> 12
- net row4: track 0.00 -> 88.4 mm, vias 0 -> 8
- net col3: track 0.00 -> 82.9 mm, vias 0 -> 8
- net col8: track 0.00 -> 81.0 mm, vias 0 -> 10
- net col4: track 0.00 -> 71.7 mm, vias 0 -> 7
- net col7: track 0.00 -> 70.8 mm, vias 0 -> 10
- net col1: track 0.00 -> 68.1 mm, vias 0 -> 6
- net row1: track 0.00 -> 67.7 mm, vias 0 -> 4
- net row3: track 0.00 -> 65.4 mm, vias 0 -> 8
- net col10: track 0.00 -> 65.4 mm, vias 0 -> 6
- net col6: track 0.00 -> 61.7 mm, vias 0 -> 10
- net col5: track 0.00 -> 59.3 mm, vias 0 -> 8
- net col2: track 0.00 -> 58.6 mm, vias 0 -> 6
- net col9: track 0.00 -> 57.0 mm, vias 0 -> 6
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Other:
- board text added: "!ワンワン!"
- board text added: "Boot"
- board text added: "Reset"
- board text added: "idawgz32 v0.0 by sporewoh"
