File: pcb/idawgz32/idawgz32.kicad_sch (KiCad schematic)
At the start: 83 parts, among them J1 USB_C_Receptacle_USB2.0, SW1 BOOT, SW1 SW_Push, SW10 SW_Push, SW11 SW_Push, SW12 SW_Push, SW13 SW_Push, SW14 SW_Push, SW15 SW_Push, SW16 SW_Push, SW17 SW_Push, SW18 SW_Push, SW19 SW_Push, SW2 RESET, SW2 SW_Push, SW20 SW_Push, SW21 SW_Push, SW22 SW_Push, SW23 SW_Push, SW24 SW_Push, SW25 SW_Push, SW26 SW_Push, SW27 SW_Push, SW28 SW_Push, SW29 SW_Push, SW3 SW_Push, SW30 SW_Push, SW31 SW_Push, SW32 SW_Push, SW4 SW_Push, SW5 SW_Push, SW6 SW_Push, SW7 SW_Push, SW8 SW_Push, SW9 SW_Push, U1 CH552T, U2 USBLC6-2SC6

Commit message: update gerbers
Parts:
- removed F1: 500mA, Fuse:Fuse_0402_1005Metric, symbol Device:Polyfuse_Small
- removed U2: USBLC6-2SC6, Package_TO_SOT_SMD:SOT-23-6, symbol Power_Protection:USBLC6-2SC6
Connections:
- net P1.0 is gone; now on net row1: U1.7 (P1.0/T2/CAP1/TIN0)
- net P1.1_A0 is gone; now on net row2: U1.8 (P1.1/T2EX/CAP2/TIN1/VBUS2/AIN0)
- net P1.2 is gone; now on net col6: U1.17 (P1.2/XI/RXD_)
- net P1.3 is gone; now on net col7: U1.16 (P1.3/XO/TXD_)
- net P1.4_CS is gone; now on net col2: U1.2 (P1.4/T2_/CAP1_/SCS/TIN2/UCC1/AIN1)
- net P1.5_MOSI is gone; now on net col3: U1.3 (P1.5/MOSI/PWM1/TIN3/UCC2/AIN2)
- net P1.6_MISO is gone; now on net col4: U1.4 (P1.6/MISO/RXD1/TIN4)
- net P1.7_SCK is gone; now on net col5: U1.5 (P1.7/SCK/TXD1/TIN5)
- net P3.0_RX is gone; now on net row4: U1.10 (P3.0/PWM1_/RXD)
- net P3.1_TX is gone; now on net row3: U1.9 (P3.1/PWM2_/TXD)
- net P3.2_A3 is gone; now on net col1: U1.1 (P3.2/TXD1_/INT0/VBUS1/AIN3)
- net P3.3 is gone; now on net col10: U1.11 (P3.3/INT1)
- net P3.4 is gone; now on net col9: U1.12 (P3.4/PWM2/RXD1_/T0)
- net P3.5 is gone; now on net col8: U1.13 (P3.5/T1)
- net PORT+ is gone; now on net UDP: J1.A6 (D+), J1.B6 (D+)
- net PORT- is gone; now on net UDM: J1.A7 (D-), J1.B7 (D-)
- net VBUS is gone; now on net VCC: J1.A4 (VBUS), J1.A9 (VBUS), J1.B4 (VBUS), J1.B9 (VBUS)
